Commit message: modified urdf to disable wrist joints and works better

File: legged_gym/resources/robots/gpr/robot.urdf (robot description, URDF)
Before this commit: robot gpr, 22 links, 21 joints
Joints:
- joint left_wrist_joint: type revolute -> fixed
- joint right_wrist_joint: type revolute -> fixed

Commit message: change the effort

File: legged_gym/resources/robots/gpr/robot.urdf (robot description, URDF)
Before this commit: robot gpr, 22 links, 21 joints
Joints:
- joint floating_base_joint: origin xyz=0 0 0 rpy=-1.57 3.14 0 -> xyz=0 0 0 rpy=-1.57 3.14 3.14
- joint left_ankle_joint: limit lower=-0.6981317 upper=0.6981317 effort=80 velocity=5 -> lower=-0.6981317 upper=0.6981317 effort=17 velocity=5
- joint left_elbow_joint: limit lower=-2.0943951 upper=2.0943951 effort=80 velocity=5 -> lower=-2.0943951 upper=2.0943951 effort=20 velocity=5
- joint left_hip_pitch_joint: limit lower=-1.5707963 upper=1.5707963 effort=80 velocity=5 -> lower=-1.5707963 upper=1.5707963 effort=40 velocity=5
- joint left_hip_roll_joint: limit lower=-0.34906585 upper=3.1852259 effort=80 velocity=5 -> lower=-0.34906585 upper=3.1852259 effort=20 velocity=5
- joint left_hip_yaw_joint: limit lower=-1.5707963 upper=1.5707963 effort=80 velocity=5 -> lower=-1.5707963 upper=1.5707963 effort=20 velocity=5
- joint left_knee_joint: limit lower=-2.0943951 upper=2.0943951 effort=80 velocity=5 -> lower=-2.0943951 upper=2.0943951 effort=40 velocity=5
- joint left_shoulder_pitch_joint: limit lower=0 upper=3.1415927 effort=80 velocity=5 -> lower=0 upper=3.1415927 effort=20 velocity=5
- joint left_shoulder_roll_joint: limit lower=-0.47996554 upper=3.6302848 effort=80 velocity=5 -> lower=-0.47996554 upper=3.6302848 effort=20 velocity=5
- joint left_shoulder_yaw_joint: limit lower=-1.5707963 upper=1.5707963 effort=80 velocity=5 -> lower=-1.5707963 upper=1.5707963 effort=20 velocity=5
- joint left_wrist_joint: limit lower=0 upper=6.2831853 effort=80 velocity=5 -> lower=0 upper=6.2831853 effort=10 velocity=5
- joint right_ankle_joint: limit lower=-0.6981317 upper=0.6981317 effort=80 velocity=5 -> lower=-0.6981317 upper=0.6981317 effort=17 velocity=5
- joint right_elbow_joint: limit lower=-2.0943951 upper=2.0943951 effort=80 velocity=5 -> lower=-2.0943951 upper=2.0943951 effort=20 velocity=5
- joint right_hip_pitch_joint: limit lower=-1.5707963 upper=1.5707963 effort=80 velocity=5 -> lower=-1.5707963 upper=1.5707963 effort=40 velocity=5
- joint right_hip_roll_joint: limit lower=-0.34906585 upper=3.1852259 effort=80 velocity=5 -> lower=-0.34906585 upper=3.1852259 effort=20 velocity=5
- joint right_hip_yaw_joint: limit lower=-1.5707963 upper=1.5707963 effort=80 velocity=5 -> lower=-1.5707963 upper=1.5707963 effort=20 velocity=5
- joint right_knee_joint: limit lower=-2.0943951 upper=2.0943951 effort=80 velocity=5 -> lower=-2.0943951 upper=2.0943951 effort=40 velocity=5
- joint right_shoulder_pitch_joint: limit lower=0 upper=3.1415927 effort=80 velocity=5 -> lower=0 upper=3.1415927 effort=20 velocity=5
- joint right_shoulder_roll_joint: limit lower=-0.47996554 upper=3.6302848 effort=80 velocity=5 -> lower=-0.47996554 upper=3.6302848 effort=20 velocity=5
- joint right_shoulder_yaw_joint: limit lower=-1.5707963 upper=1.5707963 effort=80 velocity=5 -> lower=-1.5707963 upper=1.5707963 effort=20 velocity=5
- joint right_wrist_joint: limit lower=0 upper=6.2831853 effort=80 velocity=5 -> lower=0 upper=6.2831853 effort=10 velocity=5

Commit message: get gpr working

File: legged_gym/resources/robots/gpr/robot.urdf (robot description, URDF)
Before this commit: robot gpr, 22 links, 21 joints
Joints:
- joint floating_base_joint: origin xyz=0 0 0 rpy=-1.57 3.14 3.14 -> xyz=0 0 0 rpy=-1.57 3.14 0
- joint left_elbow_joint: limit lower=-2.0943951 upper=2.0943951 effort=20 velocity=5 -> lower=-2.0943951 upper=2.0943951 effort=10 velocity=5
- joint left_shoulder_pitch_joint: limit lower=0 upper=3.1415927 effort=20 velocity=5 -> lower=0 upper=3.1415927 effort=15 velocity=5
- joint left_shoulder_roll_joint: limit lower=-0.47996554 upper=3.6302848 effort=20 velocity=5 -> lower=-0.47996554 upper=3.6302848 effort=10 velocity=5
- joint left_shoulder_yaw_joint: limit lower=-1.5707963 upper=1.5707963 effort=20 velocity=5 -> lower=-1.5707963 upper=1.5707963 effort=10 velocity=5
- joint right_elbow_joint: limit lower=-2.0943951 upper=2.0943951 effort=20 velocity=5 -> lower=-2.0943951 upper=2.0943951 effort=10 velocity=5
- joint right_shoulder_pitch_joint: limit lower=0 upper=3.1415927 effort=20 velocity=5 -> lower=0 upper=3.1415927 effort=15 velocity=5
- joint right_shoulder_roll_joint: limit lower=-0.47996554 upper=3.6302848 effort=20 velocity=5 -> lower=-0.47996554 upper=3.6302848 effort=10 velocity=5
- joint right_shoulder_yaw_joint: limit lower=-1.5707963 upper=1.5707963 effort=20 velocity=5 -> lower=-1.5707963 upper=1.5707963 effort=10 velocity=5

Commit message: change sym function with variables

File: legged_gym/resources/robots/gpr/robot.urdf (robot description, URDF)
Before this commit: robot gpr, 22 links, 21 joints
Links:
- removed link base
- added link world
Joints:
- joint floating_base_joint: parent base -> world

Commit message: change urdf

File: legged_gym/resources/robots/gpr/robot.urdf (robot description, URDF)
Before this commit: robot gpr, 22 links, 21 joints
Links:
- link left_elbow_link: geometry collision mesh filename=meshes/arm3_shell.stl; visual mesh filename=meshes/arm3_shell.stl
- link left_hand: geometry collision mesh filename=meshes/hand_shell.stl; visual mesh filename=meshes/hand_shell.stl
- link left_shoulder_pitch_link: mass 0.80769287 -> 1.10769407; geometry collision mesh filename=meshes/shoulder.stl; visual mesh filename=meshes/shoulder.stl
- link left_shoulder_roll_link: mass 0.648518913 -> 0.6485195170000001; geometry collision mesh filename=meshes/arm1_top.stl; visual mesh filename=meshes/arm1_top.stl
- link left_shoulder_yaw_link: geometry collision mesh filename=meshes/arm2_shell.stl; visual mesh filename=meshes/arm2_shell.stl
- link right_elbow_link: geometry collision mesh filename=meshes/arm3_shell2.stl; visual mesh filename=meshes/arm3_shell2.stl
- link right_hand: geometry collision mesh filename=meshes/hand_shell_2.stl; visual mesh filename=meshes/hand_shell_2.stl
- link right_shoulder_pitch_link: mass 1.10769407 -> 0.80769287; geometry collision mesh filename=meshes/shoulder_2.stl; visual mesh filename=meshes/shoulder_2.stl
- link right_shoulder_roll_link: mass 0.6485195170000001 -> 0.648518913; geometry collision mesh filename=meshes/arm1_top_2.stl; visual mesh filename=meshes/arm1_top_2.stl
- link right_shoulder_yaw_link: geometry collision mesh filename=meshes/arm2_shell_2.stl; visual mesh filename=meshes/arm2_shell_2.stl
Joints:
- joint left_elbow_joint: origin xyz=2.2775662092411332e-10 -0.026000000000000002 0.0975 rpy=-1.5707963071795865 1.5707963 0.0 -> xyz=-0.026000000000000002 0.0 -0.09799999977224338 rpy=-3.1415926071795863 -1.5707963 0.0
- joint left_shoulder_pitch_joint: origin xyz=-1.0603759e-05 0.018089564 -0.18750019 rpy=0.0 0.0 -3.1415926071795863 -> xyz=-1.0603759e-05 0.018089562050771318 0.18749980999999996 rpy=3.1415926071795868 -2.220446049250313e-15 3.1415926071795868
- joint left_shoulder_roll_joint: axis 0 0 1 -> 0 0 -1; origin xyz=0.022511964 -5.627838501275855e-05 -0.06749999993301277 rpy=1.5707963999999996 -2.220446049250313e-16 -1.5707963000000003 -> xyz=0.022511964 5.627838501275855e-05 -0.06749999993301277 rpy=1.5707963 0.0 1.5707963
- joint left_shoulder_yaw_joint: axis 0 0 -1 -> 0 0 1; origin xyz=-0.13949999999999999 0.0 0.022499999155960758 rpy=-3.1415926071795863 1.5707963 0.0 -> xyz=-0.13949999999999996 -1.4619215099879723e-09 -0.02349999915596076 rpy=-1.5707963535897926 -2.6794894969484062e-08 -1.5707962803846895
- joint right_elbow_joint: origin xyz=-0.026000000000000002 0.0 -0.09799999977224338 rpy=-3.1415926071795863 -1.5707963 0.0 -> xyz=2.2775662092411332e-10 -0.026000000000000002 0.0975 rpy=-1.5707963071795865 1.5707963 0.0
- joint right_shoulder_pitch_joint: origin xyz=-1.0603759e-05 0.018089562050771318 0.18749980999999996 rpy=3.1415926071795868 -2.220446049250313e-15 3.1415926071795868 -> xyz=-1.0603759e-05 0.018089564 -0.18750019 rpy=0.0 0.0 -3.1415926071795863
- joint right_shoulder_roll_joint: axis 0 0 -1 -> 0 0 1; origin xyz=0.022511964 5.627838501275855e-05 -0.06749999993301277 rpy=1.5707963 0.0 1.5707963 -> xyz=0.022511964 -5.627838501275855e-05 -0.06749999993301277 rpy=1.5707963999999996 -2.220446049250313e-16 -1.5707963000000003
- joint right_shoulder_yaw_joint: axis 0 0 1 -> 0 0 -1; origin xyz=-0.13949999999999996 -1.4619215099879723e-09 -0.02349999915596076 rpy=-1.5707963535897926 -2.6794894969484062e-08 -1.5707962803846895 -> xyz=-0.13949999999999999 0.0 0.022499999155960758 rpy=-3.1415926071795863 1.5707963 0.0
